File: practice-circuit/practice1.kicad_sch (KiCad schematic)
At the start: 11 parts, among them J1 Conn_02x01, SW1 SW_Push_Dual_x2, SW2 SW_Push_Dual_x2, SW3 SW_DPST_x2, U1 ATTINY85-20PU

Commit message: rah i did work on the practice footprint
Parts:
- D1: footprint (none) -> LED_SMD:LED_0201_0603Metric
- D2: footprint (none) -> LED_SMD:LED_1206_3216Metric_Pad1.42x1.75mm_HandSolder
- J1: footprint (none) -> Connector_PinHeader_1.27mm:PinHeader_2x01_P1.27mm_Vertical_SMD
- R1, R2, R4: footprint (none) -> Resistor_SMD:R_0201_0603Metric
- R3: footprint (none) -> Resistor_SMD:R_0402_1005Metric
- SW1: footprint (none) -> Button_Switch_THT:SW_Push_2P1T_Toggle_CK_PVA1xxH1xxxxxxV2
- SW2: footprint (none) -> Button_Switch_THT:SW_Push_2P1T_Toggle_CK_PVA1xxH2xxxxxxV2
- SW3: footprint (none) -> Button_Switch_THT:SW_DIP_SPSTx02_Slide_6.7x6.64mm_W7.62mm_P2.54mm_LowProfile
Changed lines of the file:
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@@
 			)
 		)
-		(property "Footprint" ""
+		(property "Footprint" "Resistor_SMD:R_0402_1005Metric"
 			(at 135.382 77.47 90)
 			(effects
@@
 			)
 		)
-		(property "Footprint" ""
+		(property "Footprint" "Resistor_SMD:R_0201_0603Metric"
 			(at 132.842 110.49 90)
 			(effects
@@
 			)
 		)
-		(property "Footprint" ""
+		(property "Footprint" "Resistor_SMD:R_0201_0603Metric"
 			(at 109.982 100.33 90)
 			(effects
@@
 			)
 		)
-		(property "Footprint" ""
+		(property "Footprint" "Button_Switch_THT:SW_Push_2P1T_Toggle_CK_PVA1xxH1xxxxxxV2"
 			(at 124.46 97.79 0)
 			(effects
@@
 			)
 		)
-		(property "Footprint" ""
+		(property "Footprint" "LED_SMD:LED_0201_0603Metric"
 			(at 124.46 64.77 0)
 			(effects
@@
 			)
 		)
-		(property "Footprint" ""
+		(property "Footprint" "Connector_PinHeader_1.27mm:PinHeader_2x01_P1.27mm_Vertical_SMD"
 			(at 205.74 93.98 0)
 			(effects
@@
 			)
 		)
-		(property "Footprint" ""
+		(property "Footprint" "Button_Switch_THT:SW_Push_2P1T_Toggle_CK_PVA1xxH2xxxxxxV2"
 			(at 101.6 88.9 0)
 			(effects
@@
 			)
 		)
-		(property "Footprint" ""
+		(property "Footprint" "Resistor_SMD:R_0201_0603Metric"
 			(at 130.302 82.55 90)
 			(effects
@@
 			)
 		)
-		(property "Datasheet" ""
+		(property "Datasheet" "kicad-embed://ATTINY85-20PU.kicad_sym"
 			(at 149.86 96.52 0)
 			(effects
@@
 			)
 		)
-		(property "Footprint" ""
+		(property "Footprint" "LED_SMD:LED_1206_3216Metric_Pad1.42x1.75mm_HandSolder"
 			(at 128.27 74.93 0)
 			(effects
@@
 			)
 		)
-		(property "Footprint" ""
+		(property "Footprint" "Button_Switch_THT:SW_DIP_SPSTx02_Slide_6.7x6.64mm_W7.62mm_P2.54mm_LowProfile"
 			(at 165.1 82.55 0)
 			(effects
@@
 	)
 	(embedded_fonts no)
+	(embedded_files
+		(file
+			(name "ATTINY85-20PU.kicad_sym")
+			(type other)
+			(data |KLUv/WBJCRURANadWyAQsx7zJvAlrehxpn4z7XQOVbVgYTMNLFEHjxURACgAQFEATwBVAFmGHr8H
+				uZc1DF/oMVZ0Sur7P47L0L/3Mozhy4EeTR6zSvayOBYSySBy6A6IOu+7veu8M/34MdAjRSeldVbH
+				+X76PdC122Fd1jzQh23Z5W4gIF5Na6lvN/pOl1Hi5r5zL++dNQdxd38djVUl9Q/dD/rGmYP+7ctz
+				3EP36TYwUZJSp6aqVtKSfGfQ4/TtRh79Bb9+7iORg7Z+TtYc6O4O2HQcZaucntnb/UD/TdbbN/zQ
+				o+Q62x/07zA425fX0cQmRnXv7cghMpEUBoiJY9D47WY8Tp+VcEGmySqsGmBQtj4qqlIr67EwCDa+
+				mrNzRsjpVb0CcqJSERCtWlE7KYMjIVFrJ1lNFL3kVCfCQ5K6DOd7t6tdkevXvE5FZ6FAifya0npm
+				Y/B30C/qgUtebslKH9/O8cX0fzLH44Y7WWM2l0zz54A29K67AUcgkCSQETt6eYAQPSwow6nSTinD
+				gIq4hJP08FDmS2mnlGFQpy8h4UsNGnoIykAmImUIKkASIr0IOuLAgIxcWZeRuc/rVn75QnXyI48C
+				G0wVYmS4QCnUmLPBP/sgGonAT+/tBnsO2PzG8goP2LQzEQ9Um4ExgclYrueIt1Ntocl8J38Kkuvy
+				k88Q31YMQ2JEGgcTMFzkMF4RPIFg5IE2MN4GgJjBwLJ0u4Veuzo2Qx50Dw==|
+			)
+			(checksum "9B882925AFBF422FF1B22C0A950CA3E8")
+		)
+	)
 )
