File: attempt2.kicad_sch (KiCad schematic)
At the start: 29 parts, among them J1 SIM_Card, U1 nRF9160-SIxA, U2 BGU7005_115

Commit message: yay
Parts:
- added C12: 50V 56p, symbol Device:C
- added C19: 56p 50V, symbol Device:C
- added C4, C5, C6, C7: 10u 6.3, symbol Device:C
- added J2, J3: U.FL-R-SMT-110, CONN1_UFL-R_HIR, symbol 2025-07-18_05-00-41:U.FL-R-SMT-110
- added JP1: SolderJumper_3_Open, symbol Jumper:SolderJumper_3_Open
- added L2: 1.5u 1.4A, symbol Device:L
- added L4: 68n 200mA, symbol Device:L
- added PS1: TPS63031DSKR, TPS63031DSKR:SON50P250X250X80-11N, symbol TPS63031DSKR:TPS63031DSKR
- added Q5: RE1C002UNTCL, DIO_RB558WMF_ROM, symbol 2025-07-16_05-21-33:RE1C002UNTCL
- added R1: 100K 1% 1/16W, symbol Device:R
- added R19: 1/16W 5% 1M, symbol Device:R
- added R2: 1M 5% 1/16W, symbol Device:R
- added R3: R, symbol Device:R
- added U4: MIC94092YC6-TR, SC-70-6_C6_MCH, symbol 2025-07-16_06-28-42:MIC94092YC6-TR
- added U5, U6: BAV74LT1, SOT-23-3_1P4X3P040_ONS, symbol 2025-07-18_04-11-05:BAV74LT1
- R5: value R -> 1/16W 1% 100k
Connections:
- net ANT: now also J2.1
- net EN: now also Q5.1 (GATE), R19.1; no longer U2.5
- net GND: now also C19.2, C4.2, C5.2, C6.2, C7.2, PS1.11 (EXP), PS1.3 (PGND), PS1.9 (GND), Q5.2 (SOURCE), R1.2, R19.2, R2.2, U4.2 (GND), U4.5 (GND); no longer U2.1, U2.2
- net GPS: now also C12.1, R3.1; no longer R5.1
- net at R3.1, U2.6: now also R3.2; no longer R5.2
- net at U2.3: no longer U1.67 (GPS)
- new net: JP1.2 (C), U5.1 (A)
- new net: C12.2, J3.1, L4.1
- new net: C19.1, L4.2, U4.1 (VOUT)
- new net: R2.1, R5.1, U5.3 (K), U6.3 (K)
- new net: U2.1, U2.2
- new net: L2.2, PS1.2 (L2)
- new net: L2.1, PS1.4 (L1)
- new net +3V3: C4.1, C5.1, PS1.1 (VOUT), PS1.10 (FB), U4.4 (VIN)
- new net COEX0/LNA_EN: R1.1, U4.6 (EN)
- new net MODE/WAKE/2: U6.1 (A)
- new net P0.31/NRF_PS_EN/2: JP1.1 (A)
- new net RTC_PS_EN/3: U6.2 (A)
- new net VSYS: C6.1, C7.1, JP1.3 (B), PS1.5 (VIN), PS1.6 (EN), PS1.7 (PS/SYNC), PS1.8 (VINA), Q5.3 (DRAIN), R5.2, U5.2 (A)
Other:
- note added: "BUCK/BOOST"
- note added: "GPS MODULE"
- note added: "UNUSED PARTS"
- moved on the sheet: R3, R4, U2

Commit message: yes
Parts:
- removed C12: C, symbol Device:C
- added C13: C, symbol Device:C
Connections:
- net GND: now also C13.2
- net GPS: now also U1.67 (GPS)
- net SDATA: now also C13.1
- net VIO: no longer U1.57 (VIO)
- net at R10.1: no longer U1.58 (SCLK)
- net at U1.59 (SDATA): no longer R9.1
Other:
- moved on the sheet: C13, C14, R10, R9

Commit message: yay pt 2
Parts:
- removed C4, C5, C6: 10u 6.3, symbol Device:C
- removed C7: C, symbol Device:C
- removed R1, R2: R, symbol Device:R
- added C11: 1u 25V, symbol Device:C
- added C13, C15: 4.7u, symbol Device:C
- added C14, C16: 0.1u, symbol Device:C
- added D1: LED, symbol Device:LED
- added D2, D3: BAT20JFILM, BAT20JFILM:SOD-323, symbol BAT20JFILM:BAT20JFILM
- added J4: USB_C_Receptacle_USB2.0_14P, symbol Connector:USB_C_Receptacle_USB2.0_14P
- added MOSFET1, MOSFET2: NX1029X_115, SOT666_1P2X1P6_NEX, symbol 2025-07-18_06-51-41:NX1029X_115
- added Q2: RE1C002UNTCL, DIO_RB558WMF_ROM, symbol 2025-07-16_05-21-33:RE1C002UNTCL
- added R11, R14, R15: R, symbol Device:R
- added R12: 2k, symbol Device:R
- added R13, R14, R17, R7: 100k, symbol Device:R
- added R15: 22k, symbol Device:R
- added R16: 33k, symbol Device:R
- added R20: 1.5k, symbol Device:R
- added R21: 5.1k, symbol Device:R
- added R4: R1k, symbol Device:R
- added R9: 1M, symbol Device:R
- added SW1, SW2, SW3: SW_Push, symbol Switch:SW_Push
- added U3: MCP73831T-2ACI_OT, MCP73831T-2ACI_OT:SOT95P280X145-5N, symbol MCP73831T-2ACI_OT:MCP73831T-2ACI_OT
- added U7: CP2102N-A02-GQFN24R, CP2102N-A02-GQFN24R:QFN50P400X400X80-25N, symbol CP2102N-A02-GQFN24R:CP2102N-A02-GQFN24R
- C1, C2, C3: value C -> 10u 6.3
- C10: value C -> 100u
- C8: value C -> 10u
- C9: value C -> 0.1u
- L1: value L -> 1.5u
Connections:
- net +3V3: now also C10.1, C2.1, C3.1, C5.1, C6.1, U1.102 (VDD1), U1.12 (VDD_GPIO), U1.22 (VDD2), R11.1, R17.1, R9.1, U3.1 (STAT)
- net ENABLE: now also R9.2
- net GND: now also C11.2, C13.1, C14.1, C15.2, C16.2, J4.A1 (GND), J4.A12 (GND), J4.B1 (GND), J4.B12 (GND), J4.S1 (SHIELD), MOSFET1.1, R12.2, R13.2, R15.2, R16.2, R20.2, R21.2, R7.2, SW2.2, SW3.1, U3.2 (VSS), U7.2 (GND), U7.25 (GND__1); no longer PS1.11 (EXP)
- net RTC_PS_EN/3: no longer U6.2 (A)
- net VSYS: now also C1.1, D2.C, Q2.1 (GATE), Q2.2 (SOURCE), R7.1, SW1.1; no longer PS1.5 (VIN), PS1.6 (EN), PS1.7 (PS/SYNC), PS1.8 (VINA), U5.2 (A)
- net at PS1.2 (L2): now also L1.2; no longer L2.2
- net at PS1.4 (L1): now also L1.1; no longer L2.1
- net at U1.32 (~{RESET}): now also R17.2, SW3.2; no longer C10.1
- removed net +3V0: C1.1, C2.1, C3.1, C5.1, C6.1, C8.1, C9.1, L1.1, U1.12 (VDD_GPIO), U1.22 (VDD2)
- new net: J4.A5 (CC1), R21.1
- new net: MOSFET1.6, MOSFET2.5, R14.2
- new net: MOSFET2.3, R14.1
- new net: R12.1, U3.5 (PROG)
- new net: D1.2 (A), R11.2
- new net: R4.1, U7.9 (~{RST})
- new net: C15.1, C16.1, U7.5 (VIO), U7.6 (VDD)
- new net: C9.1, PS1.6 (EN), PS1.7 (PS/SYNC), PS1.8 (VINA)
- new net: J4.B5 (CC2), R20.1
- new net CP2102N_VDD: R15.2, R16.1, R4.2, U7.8 (VBUS)
- new net DIFF_N: J4.A7 (D-), J4.B7 (D-), U7.4 (D-)
- new net DIFF_P: J4.A6 (D+), J4.B6 (D+), U7.3 (D+)
- new net MODE/WAKE/1: R13.1, SW1.2
- new net P0.03/D7/1: D1.1 (K)
- new net P0.20/VBAT_MEAS/2: R14.2, R15.1
- new net P0.25/VBAT_MEAS_EN/2: MOSFET1.2
- new net RESET/1: SW2.1
- new net USB_UART_RX/2: U7.21 (TXD)
- new net USB_UART_TX/2: U7.20 (RXD)
- new net VBAT: C11.1, MOSFET2.4, Q2.3 (DRAIN), R14.1, U3.3 (VBAT), U3.4 (VDD)
- new net VBUS: C13.2, C14.2, D2.A, D3.A, J4.A4 (VBUS), J4.A9 (VBUS), J4.B4 (VBUS), J4.B9 (VBUS), R15.1, U5.2 (A), U7.7 (VREGIN)
- new net VCC_5V0: D3.C
- new net VIN: C8.1, PS1.5 (VIN)
- no-connect marks 1 -> 21
Other:
- note added: "ANTENNA"
- note added: "BATTERY MEASUREMENT"
- note added: "BUCK BOOST"
- note added: "BUTTONS"
- note added: "CHARGER"
- note added: "CORNER OF DOOM :("
- note added: "LED"
- note added: "POWER CONNECTOR"
- note added: "POWER ROUTING"
- note added: "USB TO UART"
- note added: "potentially optional for clock"
- note removed: "UNUSED PARTS"
- moved on the sheet: C7, JP1, L2, PS1, Q5, R19, R2, R5, R6, R7, R8, U5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

Commit message: i cleaned the sheet
Parts:
- removed C11: 1u 25V, symbol Device:C
- removed C13 (x2), C14: C, symbol Device:C
- removed C2, C3, C7: 10u 6.3, symbol Device:C
- removed JP1: SolderJumper_3_Open, symbol Jumper:SolderJumper_3_Open
- removed L2: 1.5u 1.4A, symbol Device:L
- removed MOSFET1, MOSFET2: NX1029X_115, SOT666_1P2X1P6_NEX, symbol 2025-07-18_06-51-41:NX1029X_115
- removed Q5: RE1C002UNTCL, DIO_RB558WMF_ROM, symbol 2025-07-16_05-21-33:RE1C002UNTCL
- removed R10, R14, R15, R3 (x2), R4, R9: R, symbol Device:R
- removed R14, R7: 100k, symbol Device:R
- removed R19: 1/16W 5% 1M, symbol Device:R
- removed R5: 1/16W 1% 100k, symbol Device:R
- removed U2: BGU7005_115, BGU7005_115:PSON50P145X100X50-6N, symbol BGU7005_115:BGU7005_115
- removed U5, U6: BAV74LT1, SOT-23-3_1P4X3P040_ONS, symbol 2025-07-18_04-11-05:BAV74LT1
- C1: value 10u 6.3 -> 1u 25V
- R2: value 1M 5% 1/16W -> 100k
Connections:
- net VBAT: now also C1.1
- net VSYS: now also R2.1; no longer C1.1
- no-connect marks 21 -> 14
Other:
- note added: "CELLULAR MICROCHIP MODULE"
- note removed: "BATTERY MEASUREMENT"
- note removed: "BUCK/BOOST"
- note removed: "CORNER OF DOOM :("
- note removed: "OPTIONAL. NOT RECCOMENDED TO BE BUILT I JUST MADE IT IN CASE"
- note removed: "potentially optional for clock"
- moved on the sheet: C10, C11, C12, C13, C14, C15, C16, C19, C4, C5, C6, C8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

Commit message: asdf
Parts:
- removed D3: BAT20JFILM, BAT20JFILM:SOD-323, symbol BAT20JFILM:BAT20JFILM
- removed J2: U.FL-R-SMT-110, CONN1_UFL-R_HIR, symbol 2025-07-18_05-00-41:U.FL-R-SMT-110
- removed R13: 100k, symbol Device:R
- removed SW1, SW2: SW_Push, symbol Switch:SW_Push
- added BT1: Battery_Cell, symbol Device:Battery_Cell
- added C2: C_Polarized_Small_US, symbol Device:C_Polarized_Small_US
- added D3: LED, symbol Device:LED
- added J5: U.FL-R-SMT-110, CONN1_UFL-R_HIR, symbol 2025-07-18_05-00-41:U.FL-R-SMT-110
- added JP2: SolderJumper_2_Open, symbol Jumper:SolderJumper_2_Open
- added R3: 100k, symbol Device:R
- added R5: R, symbol Device:R
- added SW4: SW_Push, symbol Switch:SW_Push
- C1: value 1u 25V -> 1u
- R4: value R1k -> 1k
Connections:
- net +3V3: now also C11.1, U?.5 (VCC)
- net COEX0/LNA_EN: now also U1.93 (COEX0)
- net GND: now also BT1.2 (-), C2.2, D3.1 (K), R3.2
- net VBAT: now also BT1.1 (+)
- net VBUS: now also C2.1
- net VSYS: now also JP2.2 (B), SW4.1
- net at J1.7 (I/O), U?.6 (DATA2_IN): no longer J1.2 (RST)
- net at U?.8 (DATA1_IN): now also J1.2 (RST)
- net ANT: no longer names the net of R6.1, R7.1
- net ANT: now also J5.1
- net P0.03/D7/1 renamed STATUS LED
- new net: D3.2 (A), R5.2
- new net: JP2.1 (A), R5.1
- new net USER_BTN: R3.1, SW4.2
Other:
- note added: "CHANGE"
- note added: "DEBUGGING POWER LIGHT"
- note added: "GPS ANTENNA"
- note added: "NOT EXPOSED"
- note added: "TBD"
- note added: "{dblquote}ACTIVATION STATE{dblquote} POWER LIGHT"
- note removed: "GPS MODULE"
- moved on the sheet: C11, R2

Commit message: cleaned
Parts:
- added TP1, TP10, TP11, TP12, TP13, TP14, TP15, TP16, TP17, TP18, TP19, TP2, TP20, TP21, TP3, TP4, TP5, TP6, TP7, TP8, TP9: TestPoint, symbol Connector:TestPoint
- C12: value 50V 56p -> 56p
- C19: value 56p 50V -> 56p
- JP2: value SolderJumper_2_Open -> SolderJumper_Open
- L4: value 68n 200mA -> 68n
- R1: value 100K 1% 1/16W -> 100K
Connections:
- net USB_UART_RX/2 is gone; now on net USB_UART_RX: U7.21 (TXD)
- net USB_UART_TX/2 is gone; now on net USB_UART_TX: U7.20 (RXD)
- net +3V3: now also TP1.1, TP10.1, TP13.1, TP2.1, TP20.1, TP3.1, TP5.1, TP7.1
- net GND: now also C13.2, C14.2, U1.1 (GND_Shield), U1.103 (VSS), U1.11 (GND_Shield), U1.14 (GND_Shield), U1.17 (GND_Shield), U1.21 (GND_Shield), U1.27 (GND_Shield), U1.31 (GND_Shield), U1.36 (GND_Shield), U1.41 (GND_Shield), U1.44 (GND_Shield), U1.47 (GND_Shield), U1.5 (GND_Shield), U1.50 (GND_Shield), U1.52 (GND_Shield), U1.56 (GND_Shield), U1.6 (GND_Shield), U1.60 (GND_Shield), U1.62 (GND_Shield), U1.63 (GND_Shield), U1.65 (GND_Shield), U1.66 (GND_Shield), U1.68 (GND_Shield), U1.69 (GND_Shield), U1.7 (GND_Shield), U1.72 (GND_Shield), U1.74 (GND_Shield), U1.75 (GND_Shield), U1.76 (GND_Shield), U1.77 (GND_Shield), U1.78 (GND_Shield), U1.79 (GND_Shield), U1.8 (GND_Shield), U1.80 (GND_Shield), U1.81 (GND_Shield), U1.82 (GND_Shield), U1.85 (GND_Shield), U1.9 (GND_Shield), U1.90 (GND_Shield), U1.94 (GND_Shield), U1.98 (GND_Shield); no longer C13.1, C14.1
- net STATUS LED: now also U1.20 (P0.12)
- net USER_BTN: now also U1.19 (P0.11), TP19.1
- net VBAT: now also TP11.1, TP12.1
- net VBUS: now also C13.1, C14.1, TP16.1, TP17.1, TP9.1; no longer C13.2, C14.2
- net VIN: now also TP14.1
- net VSYS: now also TP18.1, TP21.1
- net at J5.1, R6.1, R7.1: now also TP4.1
- net at C12.2, J3.1, L4.1: now also TP8.1
- net at J1.1 (VCC), U1.49 (SIM_1V8): now also TP6.1
- net USB_UART_RX: now reaches U1.2 (P0.05)
- net USB_UART_TX: now reaches U1.3 (P0.06)
- net COEX0/LNA_EN renamed COEX0
- net CP2102N_VDD: no longer names the net of R15.2, R16.1, U7.8 (VBUS)
- net CP2102N_VDD: now also TP15.1; no longer R4.2
- new net VDD: R4.2
- no-connect marks 14 -> 41
Other:
- moved on the sheet: BT1, C10, C13, C14, JP2, L1, R1, R15, R16, R17, R9

Commit message: asdfklj
Parts:
- C4, C5, C6: value C -> 4.7u
Changed lines of the file:
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@@
 			)
 		)
-		(property "Value" "C"
+		(property "Value" "4.7u"
 			(at 355.6 66.0399 0)
 			(effects
@@
 			)
 		)
-		(property "Value" "C"
+		(property "Value" "4.7u"
 			(at 364.49 66.0399 0)
 			(effects
@@
 			)
 		)
-		(property "Value" "C"
+		(property "Value" "4.7u"
 			(at 346.71 66.0399 0)
 			(effects

Commit message: Initial Andrew design review
Parts:
- removed C2: C_Polarized_Small_US, symbol Device:C_Polarized_Small_US
- removed D2: BAT20JFILM, BAT20JFILM:SOD-323, symbol BAT20JFILM:BAT20JFILM
- removed Q2: RE1C002UNTCL, DIO_RB558WMF_ROM, symbol 2025-07-16_05-21-33:RE1C002UNTCL
- removed TP17, TP18: TestPoint, symbol Connector:TestPoint
- added D4: BAT20JFILM, BAT20JFILM:SOD-323, symbol BAT20JFILM:BAT20JFILM
- added R10: R, symbol Device:R
- added TP22: SWDIO, symbol Connector:TestPoint
- C14: value 0.1u -> 100n
- C16, C9: value 0.1u -> 100p
- R2: value 100k -> R
- R4: value 1k -> 10k
- TP12: value TestPoint -> SWDCLK
Connections:
- net VDD is gone; now on net VBUS: R4.2
- net VIN is gone; now on net VBUS: C8.1, PS1.5 (VIN), TP14.1
- net GND: now also R2.1; no longer R2.2
- net VBAT: now also D4.A, R10.2; no longer C1.1, TP12.1, U3.4 (VDD)
- net VBUS: now also C1.1, U3.4 (VDD), D4.C
- net VSYS: now also C10.1, C11.1, C5.1, C6.1, PS1.1 (VOUT), PS1.10 (FB), R11.1, R17.1, R9.1, TP1.1, TP13.1, TP2.1, TP20.1, TP3.1, TP5.1, TP7.1, U1.102 (VDD1), U1.12 (VDD_GPIO), U1.22 (VDD2), U4.4 (VIN), U?.5 (VCC); no longer R2.1
- net at J5.1, R6.1, R7.1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: now also R7.2, R8.1, U1.61 (ANT)
- net BAT_READ: now reaches U1.23 (AIN0/P0.13)
- net BAT_READ: now also R2.2, R10.1
- net at U1.33 (SWDCLK): now also TP12.1
- net at U1.34 (SWDIO): now also TP22.1
- removed net +3V3: C10.1, C11.1, C5.1, C6.1, PS1.1 (VOUT), PS1.10 (FB), R11.1, R17.1, R9.1, TP1.1, TP10.1, TP13.1, TP2.1, TP20.1, TP3.1, TP5.1, TP7.1, U1.102 (VDD1), U1.12 (VDD_GPIO), U1.22 (VDD2), U3.1 (STAT), U4.4 (VIN), U?.5 (VCC)
- net ENABLE: no longer names the net of R9.2, U1.101 (ENABLE)
- net STATUS LED renamed STATUS_LED
- net USB_UART_RX renamed UART_RX
- net USB_UART_TX renamed UART_TX
- new net: TP10.1, U3.1 (STAT)
- no-connect marks 41 -> 49
Other:
- note added: "# TODO: ## bake - give mia the battery sense voltage divider values - antennae things ## mia - assign footprints :) - add notes about the expected voltage/current values for things (ie. buck/boost output, VBUS/VSYS lines, etc.) - route pcb"
- note added: "VBAT = (3.0, 3.7, 4.2)V"
- note added: "VBUS = 5.1V +-0.5v"
- note removed: "POWER ROUTING"
- note removed: "TBD"
- moved on the sheet: BT1, C1, C4, C5, C6, C8, C9, R15, R16, R17, R20, R21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
